Commit message: joints now load properly

File: mobile_base_description/urdf/wheel/wheel.xacro (robot description, xacro)
@@ -12,5 +12,5 @@
     <link name="wheel_${index}">
       <visual>
-        <origin xyz="0 0 0" rpy="0 0 ${PI/2}" />
+        <origin xyz="${origin}" rpy="0 0 ${PI/2}" />
         <geometry>
           <mesh filename="$(find mobile_base_description)/meshes/mecanum_wheel.STL" scale="0.001 0.001 0.001"/>
@@ -18,5 +18,5 @@
       </visual>
       <collision>
-        <origin xyz="0 0 0" rpy="${PI/2} 0 0"/> <!--might have to rotate if wheel is flipped-->
+        <origin xyz="${origin}" rpy="${PI/2} 0 0"/> <!--might have to rotate if wheel is flipped-->
         <geometry>
           <cylinder radius="${wheel_radius}" length="${wheel_width}"/>
@@ -36,5 +36,5 @@
     <type>transmission_interface/SimpleTransmission</type>
     <joint name="wheel_${index}_joint">
-        <hardwareInterface>hardware_interface/VelocityJointInterface</hardwareInterface>
+        <hardwareInterface>hardware_interface/EffortJointInterface</hardwareInterface>
     </joint>
     <actuator name="wheel_${index}_joint_motor">
