Commit message: added wheel macro

File: mobile_base_description/urdf/base/model.xacro (robot description, xacro)
@@ -1,7 +1,40 @@
 <?xml version="1.0"?>
 <robot name="mobile_base" xmlns:xacro="http://ros.org/wiki/xacro">
+  <!--<xacro:macro name="IPS_convert" params="inches" />-->
   <xacro:property name="PI" value="3.1415926535897931" />
-  <xacro:property name="wheel_radius" value="0.050" />
-  <xacro:property name="wheel_width" value="0.0505" />
+  <xacro:property name="base_dimensions" value=".9 .7 .3" />
+  <xacro:property name="wheel_radius" value="${6*.0254}" />
+  <xacro:property name="wheel_width" value="${4*.0254}" />
+  <xacro:macro name="wheel_macro" params="index origin"> <!-- include boolean if left or right wheel-->
+    <joint name="wheel_${index}_joint" type="continuous">
+      <origin xyz="${origin}" rpy="0 0 0" />
+      <parent link="base_link"/>
+      <child link="wheel_${index}" />
+      <axis xyz="0 1 0"/>
+    </joint>
+    <link name="wheel_${index}">
+    <visual>
+      <origin xyz="0 0 0" rpy="${PI/2} 0 0" />
+      <geometry>
+        <cylinder radius="${wheel_radius}" length="${wheel_width}"/>
+      </geometry>
+    </visual>
+    <collision>
+      <origin xyz="0 0 0" rpy="${PI/2} 0 0"/> <!--might have to rotate if wheel is flipped-->
+      <geometry>
+        <cylinder radius="${wheel_radius}" length="${wheel_width}"/>
+      </geometry>
+    </collision>
+    <inertial>
+      <origin xyz="0.0 0.0 0.0" rpy="0 0 0"/>
+      <mass value="0.3844"/>
+      <!-- Inertia based on cylinder - get from CAD -->
+      <inertia
+        ixx="0.000324824" ixy="0" ixz="0"
+        iyy="0.000480000" iyz="0"
+        izz="0.000324824"/>
+    </inertial>
+  </link>
+  </xacro:macro>
   <link name="base_footprint"></link>
   <joint name="base_link_joint" type="fixed">
@@ -12,14 +45,13 @@
   <link name="base_link">
     <visual>
-      <origin xyz="0 0 0" rpy="0 0 0" />
+      <origin xyz="0 0 .2" rpy="0 0 0" />
       <geometry>
-        <box size=".9 .7 .48"/>
+        <box size="${base_dimensions}"/>
       </geometry>
-      <material name="yellow" />
     </visual>
     <collision>
       <origin xyz="0 0 0"/>
       <geometry>
-        <box size=".9 .7 .3"/>
+        <box size="${base_dimensions}"/>
       </geometry>
     </collision>
@@ -34,3 +66,7 @@
     </inertial>
   </link>
+  <xacro:wheel_macro index="0" origin=".4 .4 0"/>
+  <xacro:wheel_macro index="1" origin=".4 -.4 0"/>
+  <xacro:wheel_macro index="2" origin="-.4 -.4 0"/>
+  <xacro:wheel_macro index="3" origin="-.4 .4 0"/>
   </robot>

Commit message: added arm to base model

File: mobile_base_description/urdf/base/model.xacro (robot description, xacro)
@@ -70,3 +70,13 @@
   <xacro:wheel_macro index="2" origin="-.4 -.4 0"/>
   <xacro:wheel_macro index="3" origin="-.4 .4 0"/>
+  <!-- attach arm -->
+  <xacro:include filename="$(find kortex_description)/arms/gen3/7dof/urdf/gen3_macro.xacro"/>
+  <xacro:load_arm dof="7" vision="false" prefix="jaco_">
+    <origin xyz="0 0 0" rpy="0 0 0"/>
+  </xacro:load_arm>
+  <joint name="arm_to_base_joint" type="fixed">
+    <origin xyz="0 0 .35" rpy="0 0 0" />
+    <parent link="base_link"/>
+    <child link="jaco_base_link" />
+  </joint>
   </robot>

Commit message: moved wheel macro to new file

File: mobile_base_description/urdf/base/model.xacro (robot description, xacro)
@@ -4,37 +4,4 @@
   <xacro:property name="PI" value="3.1415926535897931" />
   <xacro:property name="base_dimensions" value=".9 .7 .3" />
-  <xacro:property name="wheel_radius" value="${6*.0254}" />
-  <xacro:property name="wheel_width" value="${4*.0254}" />
-  <xacro:macro name="wheel_macro" params="index origin"> <!-- include boolean if left or right wheel-->
-    <joint name="wheel_${index}_joint" type="continuous">
-      <origin xyz="${origin}" rpy="0 0 0" />
-      <parent link="base_link"/>
-      <child link="wheel_${index}" />
-      <axis xyz="0 1 0"/>
-    </joint>
-    <link name="wheel_${index}">
-    <visual>
-      <origin xyz="0 0 0" rpy="${PI/2} 0 0" />
-      <geometry>
-        <cylinder radius="${wheel_radius}" length="${wheel_width}"/>
-      </geometry>
-    </visual>
-    <collision>
-      <origin xyz="0 0 0" rpy="${PI/2} 0 0"/> <!--might have to rotate if wheel is flipped-->
-      <geometry>
-        <cylinder radius="${wheel_radius}" length="${wheel_width}"/>
-      </geometry>
-    </collision>
-    <inertial>
-      <origin xyz="0.0 0.0 0.0" rpy="0 0 0"/>
-      <mass value="0.3844"/>
-      <!-- Inertia based on cylinder - get from CAD -->
-      <inertia
-        ixx="0.000324824" ixy="0" ixz="0"
-        iyy="0.000480000" iyz="0"
-        izz="0.000324824"/>
-    </inertial>
-  </link>
-  </xacro:macro>
   <link name="base_footprint"></link>
   <joint name="base_link_joint" type="fixed">
@@ -43,4 +10,5 @@
     <child link="base_link" />
   </joint>
+  <!-- chassis link -->
   <link name="base_link">
     <visual>
@@ -67,8 +35,9 @@
   </link>
   <!-- attach wheels -->
-  <xacro:wheel_macro index="0" origin=".4 .4 0"/>
-  <xacro:wheel_macro index="1" origin=".4 -.4 0"/>
-  <xacro:wheel_macro index="2" origin="-.4 -.4 0"/>
-  <xacro:wheel_macro index="3" origin="-.4 .4 0"/>
+  <xacro:include filename="$(find mobile_base_description)/urdf/wheel/wheel.xacro" />
+  <xacro:wheel_macro index="0" parent="base_link" origin=".4 .4 0"/>
+  <xacro:wheel_macro index="1" parent="base_link" origin=".4 -.4 0"/>
+  <xacro:wheel_macro index="2" parent="base_link" origin="-.4 -.4 0"/>
+  <xacro:wheel_macro index="3" parent="base_link" origin="-.4 .4 0"/>
   <!-- attach arm -->
   <xacro:include filename="$(find kortex_description)/arms/gen3/7dof/urdf/gen3_macro.xacro"/>

Commit message: fixed collision vs visual base link discrepancy

File: mobile_base_description/urdf/base/model.xacro (robot description, xacro)
@@ -19,5 +19,5 @@
     </visual>
     <collision>
-      <origin xyz="0 0 0"/>
+      <origin xyz="0 0 .2"/>
       <geometry>
         <box size="${base_dimensions}"/>

Commit message: remove jaco_ prefix from arm model

File: mobile_base_description/urdf/base/model.xacro (robot description, xacro)
@@ -5,11 +5,11 @@
   <xacro:property name="base_dimensions" value=".9 .7 .3" />
   <link name="base_footprint"></link>
-  <joint name="base_link_joint" type="fixed">
+  <joint name="chassis_link_joint" type="fixed">
     <origin xyz="0 0 0.05" rpy="0 0 0" />
     <parent link="base_footprint"/>
-    <child link="base_link" />
+    <child link="chassis_link" />
   </joint>
   <!-- chassis link -->
-  <link name="base_link">
+  <link name="chassis_link">
     <visual>
       <origin xyz="0 0 .2" rpy="0 0 0" />
@@ -36,17 +36,17 @@
   <!-- attach wheels -->
   <xacro:include filename="$(find mobile_base_description)/urdf/wheel/wheel.xacro" />
-  <xacro:wheel_macro index="0" parent="base_link" origin=".4 .4 0"/>
-  <xacro:wheel_macro index="1" parent="base_link" origin=".4 -.4 0"/>
-  <xacro:wheel_macro index="2" parent="base_link" origin="-.4 -.4 0"/>
-  <xacro:wheel_macro index="3" parent="base_link" origin="-.4 .4 0"/>
+  <xacro:wheel_macro index="0" parent="chassis_link" origin=".4 .4 0"/>
+  <xacro:wheel_macro index="1" parent="chassis_link" origin=".4 -.4 0"/>
+  <xacro:wheel_macro index="2" parent="chassis_link" origin="-.4 -.4 0"/>
+  <xacro:wheel_macro index="3" parent="chassis_link" origin="-.4 .4 0"/>
   <!-- attach arm -->
   <xacro:include filename="$(find kortex_description)/arms/gen3/7dof/urdf/gen3_macro.xacro"/>
-  <xacro:load_arm dof="7" vision="false" prefix="jaco_">
+  <xacro:load_arm dof="7" vision="false" prefix="">
     <origin xyz="0 0 0" rpy="0 0 0"/>
   </xacro:load_arm>
   <joint name="arm_to_base_joint" type="fixed">
     <origin xyz="0 0 .35" rpy="0 0 0" />
-    <parent link="base_link"/>
-    <child link="jaco_base_link" />
+    <parent link="chassis_link"/>
+    <child link="base_link" /> <!-- arm base link -->
   </joint>
   <xacro:include filename="$(find mobile_base_description)/urdf/base/model.gazebo" />

Commit message: added jaco_ prefix back; experimented with commenting in launch files

File: mobile_base_description/urdf/base/model.xacro (robot description, xacro)
@@ -4,4 +4,5 @@
   <xacro:property name="PI" value="3.1415926535897931" />
   <xacro:property name="base_dimensions" value=".9 .7 .3" />
+  <xacro:property name="arm_prefix" value="jaco_" />
   <link name="base_footprint"></link>
   <joint name="chassis_link_joint" type="fixed">
@@ -42,5 +43,5 @@
   <!-- attach arm -->
   <xacro:include filename="$(find kortex_description)/arms/gen3/7dof/urdf/gen3_macro.xacro"/>
-  <xacro:load_arm dof="7" vision="false" prefix="">
+  <xacro:load_arm dof="7" vision="false" prefix="${arm_prefix}">
     <origin xyz="0 0 0" rpy="0 0 0"/>
   </xacro:load_arm>
@@ -48,6 +49,9 @@
     <origin xyz="0 0 .35" rpy="0 0 0" />
     <parent link="chassis_link"/>
-    <child link="base_link" /> <!-- arm base link -->
+    <child link="${arm_prefix}base_link" /> <!-- arm base link -->
   </joint>
   <xacro:include filename="$(find mobile_base_description)/urdf/base/model.gazebo" />
+  <!-- add in transmissions -->
+  <xacro:include filename="$(find kortex_description)/arms/gen3/7dof/urdf/gen3_transmission_macro.xacro"/>
+  <xacro:load_gazebo_arm_transmissions prefix="${arm_prefix}" />
   </robot>

Commit message: remove arm from base model

File: mobile_base_description/urdf/base/model.xacro (robot description, xacro)
@@ -40,14 +40,4 @@
   <xacro:wheel_macro index="2" parent="base_link" origin="-.4 -.4 0"/>
   <xacro:wheel_macro index="3" parent="base_link" origin="-.4 .4 0"/>
-  <!-- attach arm -->
-  <xacro:include filename="$(find kortex_description)/arms/gen3/7dof/urdf/gen3_macro.xacro"/>
-  <xacro:load_arm dof="7" vision="false" prefix="jaco_">
-    <origin xyz="0 0 0" rpy="0 0 0"/>
-  </xacro:load_arm>
-  <joint name="arm_to_base_joint" type="fixed">
-    <origin xyz="0 0 .35" rpy="0 0 0" />
-    <parent link="base_link"/>
-    <child link="jaco_base_link" />
-  </joint>
   <xacro:include filename="$(find mobile_base_description)/urdf/base/model.gazebo" />
   </robot>

Commit message: add transmissions to wheel macro

File: mobile_base_description/urdf/base/model.xacro (robot description, xacro)
@@ -43,5 +43,5 @@
   <xacro:include filename="$(find mobile_base_description)/urdf/base/model.gazebo" />
   <!-- Load wheel transmissions-->
-  <xacro:include filename="$(find mobile_base_description)/urdf/base/model_transmission.xacro" />
-  <xacro:load_base_transmissions />
+  <!-- <xacro:include filename="$(find mobile_base_description)/urdf/base/model_transmission.xacro" />
+  <xacro:load_base_transmissions /> -->
   </robot>

File: mobile_base_description/urdf/base/model_transmission.xacro (robot description, xacro)
@@ -2,13 +2,4 @@
 <robot xmlns:xacro="http://ros.org/wiki/xacro">
   <xacro:macro name="wheel_transmission" params="index">
-    <transmission name="wheel_${index}_joint_transmission">
-    <type>transmission_interface/SimpleTransmission</type>
-    <joint name="wheel_${index}_joint">
-        <hardwareInterface>hardware_interface/EffortJointInterface</hardwareInterface>
-    </joint>
-    <actuator name="wheel_${index}_joint_motor">
-        <mechanicalReduction>1</mechanicalReduction>
-    </actuator>
-    </transmission>
   </xacro:macro>
   <xacro:macro name="load_base_transmissions">

File: mobile_base_description/urdf/wheel/wheel.xacro (robot description, xacro)
@@ -33,4 +33,20 @@
       </inertial>
     </link>
+    <transmission name="wheel_${index}_joint_transmission">
+    <type>transmission_interface/SimpleTransmission</type>
+    <joint name="wheel_${index}_joint">
+        <hardwareInterface>hardware_interface/VelocityJointInterface</hardwareInterface>
+    </joint>
+    <actuator name="wheel_${index}_joint_motor">
+        <mechanicalReduction>1</mechanicalReduction>
+    </actuator>
+    </transmission>
+    <gazebo reference="wheel_${index}">
+      <mu1 value="1.0"/>
+      <mu2 value="1.0"/>
+      <kp value="10000000.0" />
+      <fdir1 value="1 0 0" />
+      <turnGravityOff>false</turnGravityOff>
+    </gazebo>
   </xacro:macro>
 </robot>

Commit message: added wheel mesh to model

File: mobile_base_description/urdf/base/model.xacro (robot description, xacro)
@@ -3,5 +3,5 @@
   <!--<xacro:macro name="IPS_convert" params="inches" />-->
   <xacro:property name="PI" value="3.1415926535897931" />
-  <xacro:property name="base_dimensions" value=".9 .7 .3" />
+  <xacro:property name="base_dimensions" value=".9 .7 .3" /> <!-- 35 by 28 by 12-->
   <link name="base_footprint"></link>
   <joint name="base_link_joint" type="fixed">

File: mobile_base_description/urdf/wheel/wheel.xacro (robot description, xacro)
@@ -1,9 +1,9 @@
 <?xml version="1.0"?>
 <robot name="mobile_base" xmlns:xacro="http://ros.org/wiki/xacro">
-  <xacro:property name="wheel_radius" value="${6*.0254}" />
-  <xacro:property name="wheel_width" value="${4*.0254}" />
+  <xacro:property name="wheel_radius" value=".0855" />
+  <xacro:property name="wheel_width" value=".1526" />
   <xacro:macro name="wheel_macro" params="index parent origin"> <!-- include boolean if left or right wheel-->
     <joint name="wheel_${index}_joint" type="continuous">
-      <origin xyz="${origin}" rpy="0 0 0" />
+      <origin xyz="${origin}" rpy="0 0 0" /><!-- TODO: figure out origin of wheel-->
       <parent link="${parent}"/>
       <child link="wheel_${index}" />
@@ -12,7 +12,7 @@
     <link name="wheel_${index}">
       <visual>
-        <origin xyz="0 0 0" rpy="${PI/2} 0 0" />
+        <origin xyz="0 0 0" rpy="0 0 ${PI/2}" />
         <geometry>
-          <cylinder radius="${wheel_radius}" length="${wheel_width}"/>
+          <mesh filename="$(find mobile_base_description)/meshes/mecanum_wheel.STL" scale="0.001 0.001 0.001"/>
         </geometry>
       </visual>

Commit message: clean up plugins

File: mobile_base_description/urdf/base/model.xacro (robot description, xacro)
@@ -1,7 +1,6 @@
 <?xml version="1.0"?>
 <robot name="mobile_base" xmlns:xacro="http://ros.org/wiki/xacro">
-  <!--<xacro:macro name="IPS_convert" params="inches" />-->
   <xacro:property name="PI" value="3.1415926535897931" />
-  <xacro:property name="base_dimensions" value=".9 .7 .3" /> <!-- 35 by 28 by 12-->
+  <xacro:property name="base_dimensions" value=".9 .7 .3" /> <!-- 35 by 28 by 12 inches-->
   <link name="base_footprint"></link>
   <joint name="chassis_link_joint" type="fixed">

Commit message: try to stick arm in base

File: mobile_base_description/urdf/base/model.xacro (robot description, xacro)
@@ -41,3 +41,37 @@
   <!-- Load gazebo file-->
   <xacro:include filename="$(find mobile_base_description)/urdf/base/model.gazebo" />
+  <!-- arm holders -->
+  <!-- <xacro:macro name="holding_block" params="index origin">
+    <link name="block_${index}">
+      <visual>
+        <origin xyz="${origin}" rpy="0 0 0" />
+        <geometry>
+          <box size=".1 .1 .1"/>
+        </geometry>
+      </visual>
+      <collision>
+        <origin xyz=".1 .1 .1"/>
+        <geometry>
+          <box size="${base_dimensions}"/>
+        </geometry>
+      </collision>
+      <inertial>
+        <origin xyz="0 0 0" rpy="0 0 0"/>
+        <mass value="1"/>
+        <inertia
+          ixx="0.018819942" ixy="0" ixz="-0.000101519"
+          iyy="0.057333716" iyz="0"
+          izz="0.074201740"/>
+      </inertial>
+    </link>
+    <joint name="block_${index}_chassis_joint" type="fixed">
+      <origin xyz="0 0 0" rpy="0 0 0" />
+      <parent link="chassis_link"/>
+      <child link="block_${index}" />
+    </joint>
+  </xacro:macro>
+  <xacro:holding_block index="1" origin=".08 .08 .35" />
+  <xacro:holding_block index="2" origin="-.08 .08 .35" />
+  <xacro:holding_block index="3" origin="-.08 -.08 .35" />
+  <xacro:holding_block index="4" origin=".08 -.08 .35" /> -->
   </robot>

Commit message: add in prismatic joint, update move demo to move in x axis

File: mobile_base_description/urdf/base/model.xacro (robot description, xacro)
@@ -3,5 +3,6 @@
   <xacro:property name="PI" value="3.1415926535897931" />
   <xacro:property name="base_dimensions" value=".9 .7 .3" /> <!-- 35 by 28 by 12 inches-->
-  <link name="base_footprint"></link>
+  <link name="world" />
+  <link name="base_footprint" />
   <joint name="chassis_link_joint" type="fixed">
     <origin xyz="0 0 0.05" rpy="0 0 0" />
@@ -41,37 +42,20 @@
   <!-- Load gazebo file-->
   <xacro:include filename="$(find mobile_base_description)/urdf/base/model.gazebo" />
-  <!-- arm holders -->
-  <!-- <xacro:macro name="holding_block" params="index origin">
-    <link name="block_${index}">
-      <visual>
-        <origin xyz="${origin}" rpy="0 0 0" />
-        <geometry>
-          <box size=".1 .1 .1"/>
-        </geometry>
-      </visual>
-      <collision>
-        <origin xyz=".1 .1 .1"/>
-        <geometry>
-          <box size="${base_dimensions}"/>
-        </geometry>
-      </collision>
-      <inertial>
-        <origin xyz="0 0 0" rpy="0 0 0"/>
-        <mass value="1"/>
-        <inertia
-          ixx="0.018819942" ixy="0" ixz="-0.000101519"
-          iyy="0.057333716" iyz="0"
-          izz="0.074201740"/>
-      </inertial>
-    </link>
-    <joint name="block_${index}_chassis_joint" type="fixed">
-      <origin xyz="0 0 0" rpy="0 0 0" />
-      <parent link="chassis_link"/>
-      <child link="block_${index}" />
+  <!-- Load world prismatic joints-->
+  <joint name="base_x_joint" type="prismatic">
+    <origin xyz="0 0 0" rpy="0 0 0" />
+    <parent link="world"/>
+    <child link="base_footprint" />
+    <axis xyz="1 0 0"/>
+    <limit effort="1000.0" lower="-0.2" upper="0.2" velocity="0.5"/>
+  </joint>
+  <transmission name="base_x_transmission">
+    <type>transmission_interface/SimpleTransmission</type>
+    <joint name="base_x_joint">
+        <hardwareInterface>hardware_interface/EffortJointInterface</hardwareInterface>
     </joint>
-  </xacro:macro>
-  <xacro:holding_block index="1" origin=".08 .08 .35" />
-  <xacro:holding_block index="2" origin="-.08 .08 .35" />
-  <xacro:holding_block index="3" origin="-.08 -.08 .35" />
-  <xacro:holding_block index="4" origin=".08 -.08 .35" /> -->
+    <actuator name="base_x_joint_motor">
+        <mechanicalReduction>1</mechanicalReduction>
+    </actuator>
+  </transmission>
   </robot>

File: mobile_base_description/urdf/wheel/wheel.xacro (robot description, xacro)
@@ -12,5 +12,5 @@
     <link name="wheel_${index}">
       <visual>
-        <origin xyz="${origin}" rpy="0 0 ${PI/2}" />
+        <origin xyz="0 0 0" rpy="0 0 ${PI/2}" />
         <geometry>
           <mesh filename="$(find mobile_base_description)/meshes/mecanum_wheel.STL" scale="0.001 0.001 0.001"/>
@@ -18,5 +18,5 @@
       </visual>
       <collision>
-        <origin xyz="${origin}" rpy="${PI/2} 0 0"/> <!--might have to rotate if wheel is flipped-->
+        <origin xyz="0 0 0" rpy="${PI/2} 0 0"/> <!--might have to rotate if wheel is flipped-->
         <geometry>
           <cylinder radius="${wheel_radius}" length="${wheel_width}"/>
@@ -33,5 +33,5 @@
       </inertial>
     </link>
-    <transmission name="wheel_${index}_joint_transmission">
+    <!-- <transmission name="wheel_${index}_joint_transmission">
     <type>transmission_interface/SimpleTransmission</type>
     <joint name="wheel_${index}_joint">
@@ -48,5 +48,5 @@
       <fdir1 value="1 0 0" />
       <turnGravityOff>false</turnGravityOff>
-    </gazebo>
+    </gazebo> -->
   </xacro:macro>
 </robot>
