Commit message: added controller descriptions and spawners to panda insert launch:

File: panda_arm/panda_insert_description/urdf/panda_insert.xacro (robot description, xacro)
@@ -10,5 +10,5 @@
   <link name="insert_link">
     <visual>
-      <origin xyz="0 0 0" rpy="0 0 0" />
+      <origin xyz="0 0 -.1" rpy="0 0 0" />
       <geometry>
         <box size=".2 .2 .2"/>
@@ -54,5 +54,5 @@
       <type>transmission_interface/SimpleTransmission</type>
       <joint name="panda_${axis_name}_joint">
-          <hardwareInterface>hardware_interface/PositionJointInterface</hardwareInterface>
+          <hardwareInterface>hardware_interface/EffortJointInterface</hardwareInterface>
       </joint>
       <actuator name="panda_${axis_name}_joint_motor">
@@ -75,5 +75,5 @@
     <type>transmission_interface/SimpleTransmission</type>
     <joint name="panda_z_rotation_joint">
-        <hardwareInterface>hardware_interface/PositionJointInterface</hardwareInterface>
+        <hardwareInterface>hardware_interface/EffortJointInterface</hardwareInterface>
     </joint>
     <actuator name="panda_z_rotation_joint_motor">
