Commit message: arm insert moves now

File: kortex_arm/kortex_insert/kortex_insert_description/urdf/kortex_insert.xacro (robot description, xacro)
@@ -1,7 +1,7 @@
 <?xml version="1.0"?>
 <robot name="kortex_insert" xmlns:xacro="http://ros.org/wiki/xacro">
-    <xacro:include filename="$(find kortex_description)/robots/gen3.xacro"/>
-<!--
-    <joint name="insert_link_joint" type="fixed">
+  <xacro:include filename="$(find kortex_description)/robots/gen3.xacro"/>
+  <link name="world" />
+  <joint name="insert_link_joint" type="fixed">
     <origin xyz="0 0 0" rpy="0 0 0" />
     <parent link="base_link"/>
@@ -10,5 +10,5 @@
   <link name="insert_link">
     <visual>
-      <origin xyz="0 0 -.2" rpy="0 0 0" />
+      <origin xyz="0 0 0" rpy="0 0 0" />
       <geometry>
         <box size=".2 .2 .2"/>
@@ -16,5 +16,5 @@
     </visual>
     <collision>
-      <origin xyz="0 0 -.2"/>
+      <origin xyz="0 0 0"/>
       <geometry>
         <box size=".2 .2 .2"/>
@@ -29,13 +29,42 @@
         izz="0.074201740"/>
     </inertial>
-  </link> -->
-    <gazebo>
-        <plugin name="kortex_controller" filename="libgazebo_ros_planar_move.so">
-            <commandTopic>cmd_vel</commandTopic>
-            <odometryTopic>odom</odometryTopic>
-            <odometryFrame>odom</odometryFrame>
-            <odometryRate>20.0</odometryRate>
-            <robotBaseFrame>base_link</robotBaseFrame>
-        </plugin>
-    </gazebo>
+  </link>
+   <!-- Load world prismatic joints-->
+  <xacro:macro name="prismatic_joint_macro" params="axis_name xyz parent child">
+    <joint name="kortex_${axis_name}_joint" type="prismatic">
+      <origin xyz="0 0 0" rpy="0 0 0" />
+      <parent link="${parent}"/>
+      <child link="${child}" />
+      <axis xyz="${xyz}"/>
+      <limit effort="1000.0" lower="-0.2" upper="0.2" velocity="0.5"/>
+    </joint>
+    <xacro:if value="${child != 'base_link'}">
+      <link name="${axis_name}_link">
+        <inertial>
+        <origin xyz="0 0 0" rpy="0 0 0" />
+        <mass value="1" />
+        <inertia
+          ixx="1.0" ixy="0.0" ixz="0.0"
+          iyy="1.0" iyz="0.0"
+          izz="1.0" />
+        </inertial>
+      </link>
+    </xacro:if>
+    <transmission name="kortex_${axis_name}_transmission">
+      <type>transmission_interface/SimpleTransmission</type>
+      <joint name="kortex_${axis_name}_joint">
+          <hardwareInterface>hardware_interface/EffortJointInterface</hardwareInterface>
+      </joint>
+      <actuator name="kortex_${axis_name}_joint_motor">
+          <mechanicalReduction>1</mechanicalReduction>
+      </actuator>
+    </transmission>
+  </xacro:macro>
+  <xacro:prismatic_joint_macro axis_name="x" xyz="1 0 0" parent="world" child="x_link"/>
+  <xacro:prismatic_joint_macro axis_name="y" xyz="0 1 0" parent="x_link" child="y_link"/>
+  <xacro:prismatic_joint_macro axis_name="z" xyz="0 0 1" parent="y_link" child="base_link"/>
+  <gazebo>
+    <plugin name="gazebo_ros_control" filename="libgazebo_ros_control.so">
+    </plugin>
+  </gazebo>
 </robot>

Commit message: spawn and move both models at the same time

File: kortex_arm/kortex_insert/kortex_insert_description/urdf/kortex_insert.xacro (robot description, xacro)
@@ -40,5 +40,5 @@
     </joint>
     <xacro:if value="${child != 'base_link'}">
-      <link name="${axis_name}_link">
+      <link name="arm_${axis_name}_link">
         <inertial>
         <origin xyz="0 0 0" rpy="0 0 0" />
@@ -61,7 +61,7 @@
     </transmission>
   </xacro:macro>
-  <xacro:prismatic_joint_macro axis_name="x" xyz="1 0 0" parent="world" child="x_link"/>
-  <xacro:prismatic_joint_macro axis_name="y" xyz="0 1 0" parent="x_link" child="y_link"/>
-  <xacro:prismatic_joint_macro axis_name="z" xyz="0 0 1" parent="y_link" child="base_link"/>
+  <xacro:prismatic_joint_macro axis_name="x" xyz="1 0 0" parent="world" child="arm_x_link"/>
+  <xacro:prismatic_joint_macro axis_name="y" xyz="0 1 0" parent="arm_x_link" child="arm_y_link"/>
+  <xacro:prismatic_joint_macro axis_name="z" xyz="0 0 1" parent="arm_y_link" child="base_link"/>
   <gazebo>
     <plugin name="gazebo_ros_control" filename="libgazebo_ros_control.so">

File: mobile_base_description/urdf/base/model.xacro (robot description, xacro)
@@ -52,5 +52,5 @@
     </joint>
     <xacro:if value="${child != 'base_footprint'}">
-      <link name="${axis_name}_link">
+      <link name="base_${axis_name}_link">
         <inertial>
         <origin xyz="0 0 0" rpy="0 0 0" />
@@ -73,6 +73,6 @@
     </transmission>
   </xacro:macro>
-  <xacro:prismatic_joint_macro axis_name="x" xyz="1 0 0" parent="world" child="x_link"/>
-  <xacro:prismatic_joint_macro axis_name="y" xyz="0 1 0" parent="x_link" child="y_link"/>
-  <xacro:prismatic_joint_macro axis_name="z" xyz="0 0 1" parent="y_link" child="base_footprint"/>
+  <xacro:prismatic_joint_macro axis_name="x" xyz="1 0 0" parent="world" child="base_x_link"/>
+  <xacro:prismatic_joint_macro axis_name="y" xyz="0 1 0" parent="base_x_link" child="base_y_link"/>
+  <xacro:prismatic_joint_macro axis_name="z" xyz="0 0 1" parent="base_y_link" child="base_footprint"/>
   </robot>

Commit message: add z rotation to model and controllers

File: kortex_arm/kortex_insert/kortex_insert_description/urdf/kortex_insert.xacro (robot description, xacro)
@@ -63,5 +63,22 @@
   <xacro:prismatic_joint_macro axis_name="x" xyz="1 0 0" parent="world" child="arm_x_link"/>
   <xacro:prismatic_joint_macro axis_name="y" xyz="0 1 0" parent="arm_x_link" child="arm_y_link"/>
-  <xacro:prismatic_joint_macro axis_name="z" xyz="0 0 1" parent="arm_y_link" child="base_link"/>
+  <xacro:prismatic_joint_macro axis_name="z" xyz="0 0 1" parent="arm_y_link" child="arm_z_link"/>
+  <!-- Load world rotation joint -->
+  <joint name="kortex_z_rotation_joint" type="continuous">
+    <origin xyz="0 0 0" rpy="0 0 0" />
+    <parent link="arm_z_link"/>
+    <child link="base_link" />
+    <axis xyz="0 0 1"/>
+    <limit effort="1000.0" lower="-0.2" upper="0.2" velocity="0.5"/>
+  </joint>
+  <transmission name="kortex_z_rotation_transmission">
+    <type>transmission_interface/SimpleTransmission</type>
+    <joint name="kortex_z_rotation_joint">
+        <hardwareInterface>hardware_interface/EffortJointInterface</hardwareInterface>
+    </joint>
+    <actuator name="kortex_z_rotation_joint_motor">
+        <mechanicalReduction>1</mechanicalReduction>
+    </actuator>
+  </transmission>
   <gazebo>
     <plugin name="gazebo_ros_control" filename="libgazebo_ros_control.so">

File: mobile_base_description/urdf/base/model.xacro (robot description, xacro)
@@ -75,4 +75,21 @@
   <xacro:prismatic_joint_macro axis_name="x" xyz="1 0 0" parent="world" child="base_x_link"/>
   <xacro:prismatic_joint_macro axis_name="y" xyz="0 1 0" parent="base_x_link" child="base_y_link"/>
-  <xacro:prismatic_joint_macro axis_name="z" xyz="0 0 1" parent="base_y_link" child="base_footprint"/>
-  </robot>
+  <xacro:prismatic_joint_macro axis_name="z" xyz="0 0 1" parent="base_y_link" child="base_z_link"/>
+  <!-- Load world rotation joint -->
+  <joint name="base_z_rotation_joint" type="continuous">
+    <origin xyz="0 0 0" rpy="0 0 0" />
+    <parent link="base_z_link"/>
+    <child link="base_footprint" />
+    <axis xyz="0 0 1"/>
+    <limit effort="1000.0" lower="-0.2" upper="0.2" velocity="0.5"/>
+  </joint>
+  <transmission name="base_z_rotation_transmission">
+    <type>transmission_interface/SimpleTransmission</type>
+    <joint name="base_z_rotation_joint">
+        <hardwareInterface>hardware_interface/EffortJointInterface</hardwareInterface>
+    </joint>
+    <actuator name="base_z_rotation_joint_motor">
+        <mechanicalReduction>1</mechanicalReduction>
+    </actuator>
+  </transmission>
+</robot>

Commit message: updated limits on prismatic joints

File: kortex_arm/kortex_insert/kortex_insert_description/urdf/kortex_insert.xacro (robot description, xacro)
@@ -37,5 +37,5 @@
       <child link="${child}" />
       <axis xyz="${xyz}"/>
-      <limit effort="1000.0" lower="-0.2" upper="0.2" velocity="0.5"/>
+      <limit effort="1000" lower="-100" upper="100" velocity="2"/>
     </joint>
     <xacro:if value="${child != 'base_link'}">

File: mobile_base_description/urdf/base/model.xacro (robot description, xacro)
@@ -49,5 +49,5 @@
       <child link="${child}" />
       <axis xyz="${xyz}"/>
-      <limit effort="1000.0" lower="-0.2" upper="0.2" velocity="0.5"/>
+      <limit effort="1000" lower="-100" upper="100" velocity="2"/>
     </joint>
     <xacro:if value="${child != 'base_footprint'}">
@@ -82,5 +82,5 @@
     <child link="base_footprint" />
     <axis xyz="0 0 1"/>
-    <limit effort="1000.0" lower="-0.2" upper="0.2" velocity="0.5"/>
+    <limit effort="1000" lower="-10" upper="10" velocity="2"/>
   </joint>
   <transmission name="base_z_rotation_transmission">

Commit message: position controllers work for insert

File: kortex_arm/kortex_insert/kortex_insert_description/urdf/kortex_insert.xacro (robot description, xacro)
@@ -54,5 +54,5 @@
       <type>transmission_interface/SimpleTransmission</type>
       <joint name="kortex_${axis_name}_joint">
-          <hardwareInterface>hardware_interface/EffortJointInterface</hardwareInterface>
+          <hardwareInterface>hardware_interface/PositionJointInterface</hardwareInterface>
       </joint>
       <actuator name="kortex_${axis_name}_joint_motor">
@@ -70,10 +70,10 @@
     <child link="base_link" />
     <axis xyz="0 0 1"/>
-    <limit effort="1000.0" lower="-0.2" upper="0.2" velocity="0.5"/>
+    <limit effort="1000.0" velocity="2"/>
   </joint>
   <transmission name="kortex_z_rotation_transmission">
     <type>transmission_interface/SimpleTransmission</type>
     <joint name="kortex_z_rotation_joint">
-        <hardwareInterface>hardware_interface/EffortJointInterface</hardwareInterface>
+        <hardwareInterface>hardware_interface/PositionJointInterface</hardwareInterface>
     </joint>
     <actuator name="kortex_z_rotation_joint_motor">

Commit message: switched kortex to use effortJointInterface like panda; tried to spawn panda at 0 0 1 (didn't work)

File: kortex_arm/kortex_insert/kortex_insert_description/urdf/kortex_insert.xacro (robot description, xacro)
@@ -54,5 +54,5 @@
       <type>transmission_interface/SimpleTransmission</type>
       <joint name="kortex_${axis_name}_joint">
-          <hardwareInterface>hardware_interface/PositionJointInterface</hardwareInterface>
+          <hardwareInterface>hardware_interface/EffortJointInterface</hardwareInterface>
       </joint>
       <actuator name="kortex_${axis_name}_joint_motor">
@@ -75,5 +75,5 @@
     <type>transmission_interface/SimpleTransmission</type>
     <joint name="kortex_z_rotation_joint">
-        <hardwareInterface>hardware_interface/PositionJointInterface</hardwareInterface>
+        <hardwareInterface>hardware_interface/EffortJointInterface</hardwareInterface>
     </joint>
     <actuator name="kortex_z_rotation_joint_motor">

File: panda_arm/panda_insert_description/urdf/panda_insert.xacro (robot description, xacro)
@@ -1,9 +1,9 @@
 <?xml version="1.0"?>
 <robot name="panda_insert" xmlns:xacro="http://ros.org/wiki/xacro">
-  <xacro:include filename="$(find franka_description)/robots/panda_arm.urdf.xacro"/>
+  <xacro:include filename="$(find franka_description)/robots/panda_arm.urdf.xacro" />
   <link name="world" />
   <joint name="insert_link_joint" type="fixed">
     <origin xyz="0 0 0" rpy="0 0 0" />
-    <parent link="panda_link0"/> <!-- I think -->
+    <parent link="panda_link0"/>
     <child link="insert_link" />
   </joint>
@@ -16,5 +16,5 @@
     </visual>
     <collision>
-      <origin xyz="0 0 0"/>
+      <origin xyz="0 0 -.1"/>
       <geometry>
         <box size=".2 .2 .2"/>
@@ -31,24 +31,22 @@
   </link>
    <!-- Load world prismatic joints-->
-  <xacro:macro name="prismatic_joint_macro" params="axis_name xyz parent child">
+  <xacro:macro name="prismatic_joint_macro" params="axis_name z:=0 axis parent child">
     <joint name="panda_${axis_name}_joint" type="prismatic">
       <origin xyz="0 0 0" rpy="0 0 0" />
       <parent link="${parent}"/>
       <child link="${child}" />
-      <axis xyz="${xyz}"/>
+      <axis xyz="${axis}"/>
       <limit effort="1000" lower="-100" upper="100" velocity="2"/>
     </joint>
-    <xacro:if value="${child != 'base_link'}">
-      <link name="arm_${axis_name}_link">
-        <inertial>
-        <origin xyz="0 0 0" rpy="0 0 0" />
-        <mass value="1" />
-        <inertia
-          ixx="1.0" ixy="0.0" ixz="0.0"
-          iyy="1.0" iyz="0.0"
-          izz="1.0" />
-        </inertial>
-      </link>
-    </xacro:if>
+    <link name="arm_${axis_name}_link">
+    <inertial>
+    <origin xyz="0 0 0" rpy="0 0 0" />
+    <mass value="1" />
+    <inertia
+        ixx="1.0" ixy="0.0" ixz="0.0"
+        iyy="1.0" iyz="0.0"
+        izz="1.0" />
+    </inertial>
+    </link>
     <transmission name="panda_${axis_name}_transmission">
       <type>transmission_interface/SimpleTransmission</type>
@@ -61,7 +59,7 @@
     </transmission>
   </xacro:macro>
-  <xacro:prismatic_joint_macro axis_name="x" xyz="1 0 0" parent="world" child="arm_x_link"/>
-  <xacro:prismatic_joint_macro axis_name="y" xyz="0 1 0" parent="arm_x_link" child="arm_y_link"/>
-  <xacro:prismatic_joint_macro axis_name="z" xyz="0 0 1" parent="arm_y_link" child="arm_z_link"/>
+  <xacro:prismatic_joint_macro axis_name="x" z="0" axis="1 0 0" parent="world" child="arm_x_link"/>
+  <xacro:prismatic_joint_macro axis_name="y" axis="0 1 0" parent="arm_x_link" child="arm_y_link"/>
+  <xacro:prismatic_joint_macro axis_name="z" axis="0 0 1" parent="arm_y_link" child="arm_z_link"/>
   <!-- Load world rotation joint -->
   <joint name="panda_z_rotation_joint" type="continuous">
