Commit message: refactored folder structure; tried to add insert to new panda package

File: panda_arm/franka_description/robots/panda_arm.xacro (robot description, xacro)
@@ -9,9 +9,9 @@
       </joint>
     </xacro:unless>
-    <link name="world"/>
+    <!-- <link name="world"/>
     <joint name="fixed" type="fixed">
       <parent link="world"/>
       <child link="${arm_id}_link0"/>
-    </joint>
+    </joint> -->
     <link name="${arm_id}_link0">
       <visual>
@@ -278,9 +278,9 @@
   </xacro:macro>
   <!-- Gazebo control plugin -->
-  <gazebo>
+  <!-- <gazebo>
     <plugin name="gazebo_ros_control" filename="libgazebo_ros_control.so">
       <robotNamespace>/panda</robotNamespace>
       <robotSimType>gazebo_ros_control/DefaultRobotHWSim</robotSimType>
     </plugin>
-  </gazebo>
+  </gazebo> -->
 </robot>

File: panda_arm/panda_insert/panda_insert_description/urdf/panda_insert.xacro (robot description, xacro)
@@ -1,5 +1,6 @@
 <?xml version="1.0"?>
 <robot name="panda_insert" xmlns:xacro="http://ros.org/wiki/xacro">
-  <xacro:include filename="$(find franka_description)/robots/panda_arm.urdf.xacro" />
+  <xacro:include filename="$(find franka_description)/robots/panda_arm.xacro" />
+  <xacro:panda_arm />
   <link name="world" />
   <joint name="insert_link_joint" type="fixed">
@@ -79,8 +80,9 @@
     </actuator>
   </transmission>
+  <!-- Gazebo control plugin -->
   <gazebo>
     <plugin name="gazebo_ros_control" filename="libgazebo_ros_control.so">
-        <robotNamespace>${arm_id}</robotNamespace>
-        <robotSimType>franka_gazebo/FrankaHWSim</robotSimType>
+      <robotNamespace>/panda</robotNamespace>
+      <robotSimType>gazebo_ros_control/DefaultRobotHWSim</robotSimType>
     </plugin>
   </gazebo>
