Commit message: tried getting new arm to work

File: panda_arm/panda_insert/panda_insert_description/urdf/panda_insert.xacro (robot description, xacro)
@@ -1,6 +1,5 @@
 <?xml version="1.0"?>
 <robot name="panda_insert" xmlns:xacro="http://ros.org/wiki/xacro">
-  <xacro:include filename="$(find franka_description)/robots/panda_arm.xacro" />
-  <xacro:panda_arm />
+  <xacro:include filename="$(find franka_description)/robots/panda_arm_hand.urdf.xacro" />
   <link name="world" />
   <joint name="insert_link_joint" type="fixed">
@@ -34,5 +33,5 @@
   <xacro:macro name="prismatic_joint_macro" params="axis_name z:=0 axis parent child">
     <joint name="panda_${axis_name}_joint" type="prismatic">
-      <origin xyz="0 0 0" rpy="0 0 0" />
+      <origin xyz="0 0 ${z}" rpy="0 0 0" />
       <parent link="${parent}"/>
       <child link="${child}" />
@@ -53,5 +52,5 @@
       <type>transmission_interface/SimpleTransmission</type>
       <joint name="panda_${axis_name}_joint">
-          <hardwareInterface>hardware_interface/EffortJointInterface</hardwareInterface>
+          <hardwareInterface>hardware_interface/PositionJointInterface</hardwareInterface>
       </joint>
       <actuator name="panda_${axis_name}_joint_motor">
@@ -60,5 +59,5 @@
     </transmission>
   </xacro:macro>
-  <xacro:prismatic_joint_macro axis_name="x" z="0" axis="1 0 0" parent="world" child="arm_x_link"/>
+  <xacro:prismatic_joint_macro axis_name="x" z="1" axis="1 0 0" parent="world" child="arm_x_link"/>
   <xacro:prismatic_joint_macro axis_name="y" axis="0 1 0" parent="arm_x_link" child="arm_y_link"/>
   <xacro:prismatic_joint_macro axis_name="z" axis="0 0 1" parent="arm_y_link" child="arm_z_link"/>
@@ -74,5 +73,5 @@
     <type>transmission_interface/SimpleTransmission</type>
     <joint name="panda_z_rotation_joint">
-        <hardwareInterface>hardware_interface/EffortJointInterface</hardwareInterface>
+        <hardwareInterface>hardware_interface/PositionJointInterface</hardwareInterface>
     </joint>
     <actuator name="panda_z_rotation_joint_motor">

Commit message: Added xyz origin control to panda insert

File: panda_arm/panda_insert/panda_insert_description/urdf/panda_insert.xacro (robot description, xacro)
@@ -1,4 +1,5 @@
 <?xml version="1.0"?>
 <robot name="panda_insert" xmlns:xacro="http://ros.org/wiki/xacro">
+  <xacro:arg name="origin" default="0 0 1" />
   <xacro:include filename="$(find franka_description)/robots/panda_arm_hand.urdf.xacro" />
   <link name="world" />
@@ -31,11 +32,11 @@
   </link>
    <!-- Load world prismatic joints-->
-  <xacro:macro name="prismatic_joint_macro" params="axis_name z:=0 axis parent child">
+  <xacro:macro name="prismatic_joint_macro" params="axis_name origin:='0 0 0' axis parent child">
     <joint name="panda_${axis_name}_joint" type="prismatic">
-      <origin xyz="0 0 ${z}" rpy="0 0 0" />
+      <origin xyz="${origin}" rpy="0 0 0" />
       <parent link="${parent}"/>
       <child link="${child}" />
       <axis xyz="${axis}"/>
-      <limit effort="1000" lower="-100" upper="100" velocity="2"/>
+      <limit effort="1000" lower="-1000" upper="1000" velocity="2"/>
     </joint>
     <link name="arm_${axis_name}_link">
@@ -59,5 +60,5 @@
     </transmission>
   </xacro:macro>
-  <xacro:prismatic_joint_macro axis_name="x" z="1" axis="1 0 0" parent="world" child="arm_x_link"/>
+  <xacro:prismatic_joint_macro axis_name="x" origin="$(arg origin)" axis="1 0 0" parent="world" child="arm_x_link"/>
   <xacro:prismatic_joint_macro axis_name="y" axis="0 1 0" parent="arm_x_link" child="arm_y_link"/>
   <xacro:prismatic_joint_macro axis_name="z" axis="0 0 1" parent="arm_y_link" child="arm_z_link"/>
